File: Global_Val_Sen/Global_Val_Sen.kicad_pcb (KiCad board)
At the start: 2 copper layers, 148 x 39 mm, 63 parts, among them IC2 DW01A, Q1 FS8205A, Q2 IRF7303, U1 CPU1, U2 TP4056

Commit message: actualizacion sensor Cod &PCB
Connections:
- A1 pad 3: SCL0 -> SDA0
- A1 pad 4: SDA0 -> SCL0
- A2 pad 2: Net-(A2-Pad2) -> S3.3v
- A2 pad 3: Net-(A2-Pad3) -> SGND
- JD_sen1 pad 10: Net-(JD_sen1-Pad10) -> SGND
- JD_sen1 pad 11: Net-(JD_sen1-Pad11) -> S3.3v
- JD_sen1 pad 12: Net-(JD_sen1-Pad12) -> +5V
- Q2 pad 5: Net-(A2-Pad3) -> SGND
- Q2 pad 6: Net-(A2-Pad3) -> SGND
Routing:
- net SGND: track 0.00 -> 19.3 mm
- net Net-(A2-Pad3): track 11.0 -> 0.00 mm
- net S3.3v: track 0.00 -> 8.57 mm
- net +5V: track 96.7 -> 101.7 mm
- net SDA0: track 52.4 -> 51.2 mm
- removed copper zone on B.Cu, net (none)
